File: USB-C_PD_Connector/elec/layout/default/usb-c-pd-connector.kicad_pcb (KiCad board)
At the start: 2 copper layers, 40 x 20 mm, 5 parts

Commit message: added 'designed by glowingkitty' silkscreen
Parts:
- moved REF** 11.8 mm to (102.7, 59.4)
Other:
- board text added: "designed by glowingkitty"
