File: big-cap/elec/layout/default/big-cap.kicad_pcb (KiCad board)
At the start: 2 copper layers, 40 x 20 mm, 5 parts

Commit message: added 'designed by glowingkitty' silkscreen
Parts:
- moved REF** 11.3 mm to (148.0, 84.7)
Other:
- board text added: "designed by glowingkitty"

Commit message: adapted pin header position and removed silkscreen
Parts:
- turned U1 to 180 degrees
