File: usb-to-serial/elec/layout/default/usb-to-serial.kicad_pcb (KiCad board)
At the start: 2 copper layers, 40 x 40 mm, 13 parts

Commit message: finished usb to serial layout
Other:
- board text added: "bit.ly/4cyi2lz"
- board text removed: "bit.ly/...."
